File: Greaseweazle F1 Plus 3.5/Greaseweazle F1 Plus 3.5.kicad_pcb (KiCad board)
At the start: 2 copper layers, 170.2 x 100 mm, 106 parts, among them CN1 Floppy Data, J1 USB B, J10 Conn_01x03, J11 Conn_01x03, J12 Display Port, J13 Display Port, J14 SD Module, J15 SD Module, J16 SD Module, J2 USB Header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

Commit message: Some silk screen updates
Changed lines of the file:
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@@
   (general
     (thickness 1.6)
-    (drawings 421)
+    (drawings 423)
     (tracks 1153)
     (zones 0)
@@
     (44 Edge.Cuts user)
     (45 Margin user)
-    (46 B.CrtYd user hide)
+    (46 B.CrtYd user)
     (47 F.CrtYd user)
-    (49 F.Fab user hide)
+    (49 F.Fab user)
   )
   (setup
@@
     )
   )
+  (dimension 94.005414 (width 0.254) (layer Dwgs.User)
+    (gr_text "94.005 mm" (at 234.604393 100.928205 270.0309623) (layer Dwgs.User)
+      (effects (font (size 1 1) (thickness 0.15)))
+    )
+    (feature1 (pts (xy 190.0428 147.955) (xy 233.812213 147.931347)))
+    (feature2 (pts (xy 189.992 53.9496) (xy 233.761413 53.925947)))
+    (crossbar (pts (xy 233.174993 53.926264) (xy 233.225793 147.931664)))
+    (arrow1a (pts (xy 233.225793 147.931664) (xy 232.638764 146.805477)))
+    (arrow1b (pts (xy 233.225793 147.931664) (xy 233.811605 146.804844)))
+    (arrow2a (pts (xy 233.174993 53.926264) (xy 232.589181 55.053084)))
+    (arrow2b (pts (xy 233.174993 53.926264) (xy 233.762022 55.052451)))
+  )
+  (dimension 69.977005 (width 0.254) (layer Dwgs.User)
+    (gr_text "69.977 mm" (at 154.999487 42.906452 0.02079701524) (layer Dwgs.User)
+      (effects (font (size 1 1) (thickness 0.15)))
+    )
+    (feature1 (pts (xy 189.992 53.9496) (xy 189.988284 43.711331)))
+    (feature2 (pts (xy 120.015 53.975) (xy 120.011284 43.736731)))
+    (crossbar (pts (xy 120.011497 44.323152) (xy 189.988497 44.297752)))
+    (arrow1a (pts (xy 189.988497 44.297752) (xy 188.862206 44.884582)))
+    (arrow1b (pts (xy 189.988497 44.297752) (xy 188.86178 43.71174)))
+    (arrow2a (pts (xy 120.011497 44.323152) (xy 121.138214 44.909164)))
+    (arrow2b (pts (xy 120.011497 44.323152) (xy 121.137788 43.736322)))
+  )
   (gr_text SWD (at 214.503 129.54 90) (layer B.SilkS)
     (effects (font (size 2 2) (thickness 0.125)) (justify mirror))
@@
   (gr_line (start 193.675 139.573) (end 202.311 139.7) (layer F.SilkS) (width 0.12))
   (gr_line (start 193.675 137.16) (end 202.311 137.16) (layer F.SilkS) (width 0.12))
-  (gr_circle (center 75.438 127) (end 75.538 127) (layer F.SilkS) (width 0.2))
-  (gr_circle (center 75.438 109.982) (end 75.538 109.982) (layer F.SilkS) (width 0.2))
+  (gr_circle (center 75.438 127) (end 75.588 127) (layer F.SilkS) (width 0.3))
+  (gr_circle (center 75.438 109.982) (end 75.588 109.982) (layer F.SilkS) (width 0.3))
   (gr_line (start 73.66 137.795) (end 86.995 137.795) (layer F.SilkS) (width 0.12))
   (gr_line (start 73.66 105.41) (end 86.995 105.41) (layer F.SilkS) (width 0.12))
@@
   (gr_circle (center 147.32 61.468) (end 147.52 61.468) (layer F.SilkS) (width 0.4))
   (gr_circle (center 95.377 58.547) (end 95.577 58.547) (layer F.SilkS) (width 0.4))
-  (gr_circle (center 86.233 77.343) (end 86.333 77.343) (layer F.SilkS) (width 0.2))
-  (gr_circle (center 83.439 68.707) (end 83.539 68.707) (layer F.SilkS) (width 0.2))
-  (gr_circle (center 74.676 74.803) (end 74.776 74.803) (layer F.SilkS) (width 0.2))
-  (gr_circle (center 76.454 57.404) (end 76.554 57.404) (layer F.SilkS) (width 0.2))
+  (gr_circle (center 86.233 77.343) (end 86.383 77.343) (layer F.SilkS) (width 0.3))
+  (gr_circle (center 83.439 68.707) (end 83.589 68.707) (layer F.SilkS) (width 0.3))
+  (gr_circle (center 74.676 74.803) (end 74.826 74.803) (layer F.SilkS) (width 0.3))
+  (gr_circle (center 76.454 57.404) (end 76.604 57.404) (layer F.SilkS) (width 0.3))
   (gr_text "Reverse\nPolarity\nProtection" (at 73.914 67.564) (layer F.SilkS)
     (effects (font (size 0.6 0.6) (thickness 0.1)) (justify left))
