File: Greaseweazle F1 Plus Gotek/Greaseweazle F1 Plus Gotek.kicad_pcb (KiCad board)
At the start: 2 copper layers, 114.1 x 94.7 mm, 88 parts, among them CN1 Floppy Data, J1 SWD, J2 Floppy Power, J3 Programming Port, J4 USB B, J5 Boot Header, J6 Display Connector, J7 SD Module, J8 SWD, J9 SD Module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

Commit message: Some silk screen updates
Other:
- board text removed: "Firmware Update"
- board text removed: "{"
